File: BLDC Motor Rev 2/BLDC Motor.sch (EAGLE design)
At the start: 62 parts, among them IC1 7805TV, IC2 7815TV, Q12 IRFS, Q15 IRFS, Q18 IRFS, Q3 IRFS, Q6 IRFS, Q9 IRFS, U1 ATMEGA328P_TQFP, Y1 16M

Commit message: Final board design, added test arduino code
Parts:
- added JP3: (no value), SparkFun:M07
Connections:
- net GND: now also JP3.1
- net MOSI: now also JP3.6
- net PULSE1: now also JP3.7
- net PULSE2: now also JP3.2
- net PULSE3: now also JP3.3
- net PULSE4: now also JP3.4
- net PULSE5: now also JP3.5
Other:
- note added: "Small signal mosfets are all 2n7000"
Changed lines of the file:
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@@
 <part name="GND25" library="SparkFun" deviceset="GND" device=""/>
 <part name="GND29" library="SparkFun" deviceset="GND" device=""/>
+<part name="JP3" library="SparkFun" deviceset="M07" device=""/>
+<part name="GND20" library="SparkFun" deviceset="GND" device=""/>
 </parts>
 <sheets>
 <sheet>
 <plain>
-<text x="187.96" y="254" size="1.778" layer="91">Supply Voltage: 22.2V</text>
+<text x="187.96" y="254" size="1.778" layer="97">Supply Voltage: 22.2V</text>
 <text x="325.12" y="15.24" size="1.778" layer="91">2</text>
 <text x="330.2" y="5.08" size="1.778" layer="91">Forrest Kaminski</text>
+<text x="132.08" y="127" size="1.778" layer="97">Small signal mosfets are all 2n7000</text>
 </plain>
 <instances>
@@
 <instance part="GND25" gate="1" x="139.7" y="71.12"/>
 <instance part="GND29" gate="1" x="127" y="66.04"/>
+<instance part="JP3" gate="G$1" x="241.3" y="233.68"/>
+<instance part="GND20" gate="1" x="251.46" y="223.52"/>
 </instances>
 <busses>
@@
 <pinref part="GND29" gate="1" pin="GND"/>
 </segment>
+<segment>
+<pinref part="JP3" gate="G$1" pin="1"/>
+<wire x1="246.38" y1="228.6" x2="251.46" y2="228.6" width="0.1524" layer="91"/>
+<wire x1="251.46" y1="228.6" x2="251.46" y2="226.06" width="0.1524" layer="91"/>
+<pinref part="GND20" gate="1" pin="GND"/>
+</segment>
 </net>
 <net name="N$1" class="0">
@@
 <pinref part="R17" gate="G$1" pin="2"/>
 </segment>
+<segment>
+<pinref part="JP3" gate="G$1" pin="7"/>
+<wire x1="246.38" y1="243.84" x2="248.92" y2="243.84" width="0.1524" layer="91"/>
+<label x="248.92" y="243.84" size="1.778" layer="95"/>
+</segment>
 </net>
 <net name="N$17" class="0">
@@
 <pinref part="R20" gate="G$1" pin="2"/>
 </segment>
+<segment>
+<pinref part="JP3" gate="G$1" pin="2"/>
+<wire x1="246.38" y1="231.14" x2="248.92" y2="231.14" width="0.1524" layer="91"/>
+<label x="248.92" y="231.14" size="1.778" layer="95"/>
+</segment>
 </net>
 <net name="PULSE3" class="0">
@@
 <pinref part="R21" gate="G$1" pin="2"/>
 </segment>
+<segment>
+<pinref part="JP3" gate="G$1" pin="3"/>
+<wire x1="246.38" y1="233.68" x2="248.92" y2="233.68" width="0.1524" layer="91"/>
+<label x="248.92" y="233.68" size="1.778" layer="95"/>
+</segment>
 </net>
 <net name="N$20" class="0">
@@
 <pinref part="R22" gate="G$1" pin="2"/>
 </segment>
+<segment>
+<pinref part="JP3" gate="G$1" pin="4"/>
+<wire x1="246.38" y1="236.22" x2="248.92" y2="236.22" width="0.1524" layer="91"/>
+<label x="248.92" y="236.22" size="1.778" layer="95"/>
+</segment>
 </net>
 <net name="PULSE5" class="0">
@@
 <pinref part="R19" gate="G$1" pin="2"/>
 </segment>
+<segment>
+<pinref part="JP3" gate="G$1" pin="5"/>
+<wire x1="246.38" y1="238.76" x2="248.92" y2="238.76" width="0.1524" layer="91"/>
+<label x="248.92" y="238.76" size="1.778" layer="95"/>
+</segment>
 </net>
 <net name="MOSI" class="0">
@@
 <pinref part="R18" gate="G$1" pin="2"/>
 </segment>
-</net>
+<segment>
+<pinref part="JP3" gate="G$1" pin="6"/>
+<wire x1="246.38" y1="241.3" x2="248.92" y2="241.3" width="0.1524" layer="91"/>
+<label x="248.92" y="241.3" size="1.778" layer="95"/>
+</segment>
+</net>
